File: power.kicad_sch (KiCad schematic)
At the start: 56 parts, among them J1 PWR + CAN harness, Q1 100V 6.8mOhm N-ch, U1 LM74700-Q1, U2 LM5164 (5V), U3 LM5164 (3V3)

Commit message: Schematic: power symbols and readable text placement (items 1-2 of 5)
The schematic was a netlist drawn as a picture: 486 global labels for 108
nets, roughly four per net, every part an island with a name flag on each
pin and no wires between anything. You could not trace a circuit by eye.
That is a fair description of a document that fails at the one thing a
schematic is for, and it is on me -- the generator was built to produce a
correct netlist and the drawing was an afterthought.

Two of the five agreed fixes are in:

Rails are power symbols. GND, +3V3, +5V, +5VS, +VBAT, VBUS and SD_VDD now
carry a proper power symbol instead of a net-name label -- 190 of them,
taking the label count from 486 to 296. Where KiCad has no stock symbol
for a rail a generic one is instantiated with its Value overridden, which
is how KiCad names a power net; validate.py re-extracts through KiCad and
compares node-for-node, so a wrong guess there would fail the build rather
than quietly merge two rails. PWR_FLAG keeps a label: pairing it with a
power symbol makes an island of two symbols that declares a rail and
connects to nothing visible.

Text no longer collides. Labels were all justified left, so any label
pointing back at its own component ran its text over the body -- RON_5V
across R4, SW_5V across L1; they now justify away from the part.
Reference and value sat hard against the symbol, so a pin leaving the top
or bottom put its stub and power symbol straight through them: "LM5164
(5V)" printed through the GND symbol under U2. Both now clear the stub,
and the row height accounts for it so the clearance does not just push
the collision into the next row. Power symbol references are hidden, as
they are in every schematic.

Also fixed: the packer wrapped on height but never on width, so the power
sheet silently ran off the 420 mm page -- two symbols landed at x = 422.9
where ERC reported them unconnected and nothing else complained. It now
fails loudly.

Items 3-5 (real hierarchy, w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
Parts:
- added C18: 22uF, Capacitor_SMD:C_1206_3216Metric, symbol Device:C
- added C19: 100nF, Capacitor_SMD:C_0805_2012Metric, symbol Device:C
- added C20: 10uF, Capacitor_SMD:C_1206_3216Metric, symbol Device:C
- added TP6: +5VS, TestPoint:TestPoint_Pad_D1.5mm, symbol Connector:TestPoint
- added TP7: GND, TestPoint:TestPoint_Pad_D1.5mm, symbol Connector:TestPoint
- C1: value 1uF 50V -> 1uF; Voltage (none) -> 50V
- C10: value 100nF 16V -> 22uF; footprint Capacitor_SMD:C_0805_2012Metric -> Capacitor_SMD:C_1206_3216Metric; Voltage (none) -> 16V
- C11: value 2.2nF 50V -> 22uF; footprint Capacitor_SMD:C_0805_2012Metric -> Capacitor_SMD:C_1206_3216Metric; Note Bootstrap: datasheet-mandated 2.2nF X7R, do not increase -> (none); Voltage (none) -> 16V
- C12: value 3.3nF 50V -> 100nF; Note Ramp capacitor CA -> (none); Voltage (none) -> 16V
- C13: value 270pF 50V -> 10nF; Note Ramp coupling capacitor CB -> EN noise immunity, as for the 5V rail; Voltage (none) -> 100V
- C14: value 22uF 6.3V -> 2.2nF; footprint Capacitor_SMD:C_1206_3216Metric -> Capacitor_SMD:C_0805_2012Metric; Note (none) -> Bootstrap: datasheet-mandated 2.2nF X7R, do not increase; Voltage (none) -> 50V
- C15: value 22uF 6.3V -> 3.3nF; footprint Capacitor_SMD:C_1206_3216Metric -> Capacitor_SMD:C_0805_2012Metric; Note (none) -> Ramp capacitor CA; Voltage (none) -> 50V
- C16: value 100nF 16V -> 270pF; Note (none) -> Ramp coupling capacitor CB; Voltage (none) -> 50V
- C17: value 10uF 16V -> 22uF; Voltage (none) -> 16V
- C2: value 100uF 100V -> 100nF; footprint Capacitor_SMD:CP_Elec_10x10.5 -> Capacitor_SMD:C_0805_2012Metric; MPN Nichicon UCD2A101MNL1GS -> (none); Note Bulk hold-up; any 100uF >=80V SMD electrolytic on a 10x10.5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 -> LM74700 ANODE input capacitor: the datasheet requires a min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; Voltage (none) -> 100V
- C3: value 10uF 100V -> 100uF; footprint Capacitor_SMD:C_1206_3216Metric -> Capacitor_SMD:CP_Elec_10x10.5; MPN (none) -> Nichicon UCD2A101MNL1GS; Note Switcher input bypass -> Bulk hold-up; any 100uF >=80V SMD electrolytic on a 10x10.5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; Voltage (none) -> 100V
- C4: value 100nF 100V -> 10uF; footprint Capacitor_SMD:C_0805_2012Metric -> Capacitor_SMD:C_1206_3216Metric; Note HF bypass -> Switcher input bypass; Voltage (none) -> 100V
- C5: value 2.2nF 50V -> 100nF; Note Bootstrap: datasheet mandates exactly 2.2nF X7R -- a larger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 -> HF bypass; Voltage (none) -> 100V
- C6: value 3.3nF 50V -> 10nF; Note Ramp capacitor CA -> EN sits on a bare 100k to VBAT; this keeps a high-impedance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; Voltage (none) -> 100V
- C7: value 270pF 50V -> 2.2nF; Note Ramp coupling capacitor CB -> Bootstrap: datasheet mandates exactly 2.2nF X7R -- a larger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; Voltage (none) -> 50V
- C8: value 22uF 16V -> 3.3nF; footprint Capacitor_SMD:C_1206_3216Metric -> Capacitor_SMD:C_0805_2012Metric; Note (none) -> Ramp capacitor CA; Voltage (none) -> 50V
- C9: value 22uF 16V -> 270pF; footprint Capacitor_SMD:C_1206_3216Metric -> Capacitor_SMD:C_0805_2012Metric; Note (none) -> Ramp coupling capacitor CB; Voltage (none) -> 50V
- D1: value SMCJ33A -> SMCJ40A; symbol Device:D_TVS -> Device:D_Zener; MPN Littelfuse SMCJ33A -> Littelfuse SMCJ40A; Note 33V standoff / 53.3V clamp @ 1500W: absorbs ISO 7637-2 puls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 -> 40V standoff / 64.5V clamp @ 1500W: absorbs ISO 7637-2 puls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
- D3: value SMAJ5.0A -> SMAJ6.0A; symbol Device:D_TVS -> Device:D_Zener; MPN Littelfuse SMAJ5.0A -> Littelfuse SMAJ6.0A; Note Clamps harness-injected transients on the sensor 5V -> Clamps harness-injected transients on the sensor 5V. 6.0V s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
- R2: value 25.5k -> 44.2k; Note UVLO lower leg -> board enables at ~5.9V -> UVLO lower leg. Ratio 0.3065 against V_EN_IH 1.06/2.0/2.6V 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
- TP1: value +VBAT -> PG_5V
- TP2: value +5V -> PG_3V3
- TP3: value +3V3 -> +VBAT
- TP4: value +5VS -> +5V
- TP5: value GND -> +3V3
Connections:
- net +3V3: now also C15.2, C17.1, TP5.1, C18.1, C19.1; no longer C12.2, C14.1, C15.1, C16.1, TP3.1
- net +5V: now also C11.1, C12.1, C8.2, TP4.1; no longer C6.2, C8.1, C9.1, TP2.1
- net +5VS: now also C20.1, TP6.1; no longer C17.1, TP4.1
- net +VBAT: now also C5.1, TP3.1; no longer C2.1, TP1.1
- net BST_3V3: now also C14.1; no longer C11.1
- net BST_5V: now also C7.1; no longer C5.1
- net EN_3V3: now also C13.1
- net EN_5V: now also C6.1
- net FB_3V3: now also C16.2; no longer C13.2
- net FB_5V: now also C9.2; no longer C7.2
- net GND: now also C11.2, C12.2, C13.2, C5.2, C6.2, C18.2, C19.2, C20.2, TP7.1; no longer C14.2, C15.2, C16.2, C8.2, C9.2, TP5.1
- net PG_3V3: now also TP2.1
- net PG_5V: now also TP1.1
- net RAMP_3V3: now also C15.1, C16.1; no longer C12.1, C13.1
- net RAMP_5V: now also C8.1, C9.1; no longer C6.1, C7.1
- net SW_3V3: now also C14.2; no longer C11.2
- net SW_5V: now also C7.2; no longer C5.2
- net VBAT_FB: now also C2.1
Other:
- moved on the sheet: C1, C10, C11, C12, C13, C14, C15, C16, C17, C2, C3, C4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

Commit message: Rev B is fully routed: zero DRC errors, nothing unconnected
84 x 84 mm, 1447 tracks, 258 vias, 179 footprints, 106 nets.

The last few connections were never routing problems. Each one was a part
sited away from the net it belongs to, and the autorouter reporting "no
path at any width" was telling the truth:

  +5VS  the sensor rail's source (PF1/FB2/D3) sat on the right beside the
        WS2812 header while everything it feeds -- the sensor harness and
        all four channel pull-ups -- is on the left. The net existed as
        two complete halves with a 45 mm gap through buck islands and the
        SD socket. Moved the source to the harness side.
  IO46  the strapping pull-downs were parked in the bottom band while
        IO3/IO45/IO46 run from the module's south pads to J7 at the top
        left, so R29 needed a trace the length of the board to reach its
        own net. Moved them under the module's south pads.

Adding router passes had never touched either. Moving the parts fixed
both immediately -- worth remembering next time a net "cannot be routed".

Also in this pass:

  - One LED. D6 (amber) and D7 (blue) and their resistors are gone; D4
    green stays on +3V3, which is the right rail to watch because it only
    lights if the whole chain came through -- battery, ideal diode, both
    converters. That also retires review item 11.2.10, the blue emitter
    that would have been near-invisible on a 3.288 V rail.
  - J7 grows to six pins: the three strapping pins, the two GPIOs freed
    by the LEDs (IO15/IO16), and a ground pin. The missing ground was
    review item 13.4.13.
  - USB_CC1 gets a Fine netclass at 0.2 mm. There is no route at 0.25 mm
    -- the USB-C pads are on 0.5 mm pitch and will not pass it -- and CC
    carries under a milliamp through a 5.1k pull-down.
  - build_board.py takes a lock. Two builds sharing the board file is how
    one run died at "Specctra session import failed" after ten minutes,
    when a second build regenerated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
Parts:
- D4: Note Power indicator -> The board's only LED: +3V3 is up, so the whole supply chain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
Changed lines of the file:
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@@
       (effects (font (size 1.27 1.27)) hide)
     )
-    (property "Note" "Power indicator" (at 284.48 154.4 0)
+    (property "Note" "The board's only LED: +3V3 is up, so the whole supply chain came through -- battery, ideal diode, and both converters" (at 284.48 154.4 0)
       (effects (font (size 1.27 1.27)) hide)
     )
