File: power.kicad_sch (KiCad schematic)
At the start: 76 parts, among them J1 PWR + CAN harness, Q1 IPD068N10, Q2 AO3401A, Q3 2N7002, U1 LM74700-Q1, U2 TLV431A, U3 LM5164 (5V), U4 LM5164 (3V3)

Commit message: Board change: termination off by default, 0-5 V sensors by default, 2x330 uF
Three defaults changed in gen/generate_schematic.py, then the whole chain
regenerated: schematic, board, fab, plots. Schematic is ERC-clean at 206
components / 114 nets; the board rebuilt to 0 DRC violations and 0
unconnected; fab BOM and CPL agree at 178 designators.

CAN termination now ships OFF. JP1 moves from SolderJumper-2_Bridged to
_Open. The board was shipping terminated, matching the Autosport Labs
convention, but the common case here is plugging into a vehicle bus that
is already terminated at both ends — where a third 120 ohm takes the pair
to about 40 ohm and can stop the bus working. Defaulting on made that an
easy mistake; defaulting off means there is nothing to remember before
plugging into a car, and bridging JP1 is a deliberate act for a bench bus
where this board is an end node.

Analog channels now ship in the 0-5 V range. The four RANGE jumpers move
from SolderJumper-3_Open to _Bridged12, closing the 15k leg. They were
shipping fully open, which is no divider at all, so a 5 V sensor needed a
jumper somebody had to remember to fit — and the firmware's DIVIDER_GAIN
of 1.7334 assumed the 0-5 V ratio, so an unfitted jumper read 73 % high.
Board and firmware defaults now agree out of the box.

Ride-through bank 540 -> 760 uF. C6/C7 go 220 -> 330 uF in CP_Elec_16x22.
That footprint is identical to the 16x17.5 it replaces in every copper,
courtyard, silk and fab layer — only the 3D can is 4.5 mm taller — so the
extra 220 uF costs nothing but enclosure height, and the routed board did
not have to move for it.

It is not free everywhere: inrush I2t is linear in C, so the 2 A fuse's
margin drops from ~5x to ~3.6x. Noted in the generator next to the value
so the next person to grow the bank sees it.

ngspice is not installed here, so the new hold-up figures (152 / 75 ms,
from 108 / 53) are SCALED, not measured — hold-up is linear in C for a
constant-power load over a fixed window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
Parts:
- C6, C7: value 220uF -> 330uF; footprint Capacitor_SMD:CP_Elec_16x17.5 -> Capacitor_SMD:CP_Elec_16x22; Note Power-fail ride-through. With the sensor rail shed and the LEDs off the board draws about 0.35 W here, so the bank holds the rails up for roughly 70 ms -- enough to finish the block in flight and close the file. Any 220uF >=80V on a 16x17.5 land works; match in the JLC catalogue at order. Pin 1 is + -> Power-fail ride-through. With the sensor rail shed and the LEDs off the board draws about 0.35 W here, so the bank holds the rails up long enough to finish the block in flight and close the file. 16x22 rather than 16x17.5: the two footprints are identical in every copper and courtyard layer -- only the can is 4.5 mm taller -- so the extra 220 uF costs nothing but enclosure height. Any 330uF >=80V on a 16 mm land works; match in the JLC catalogue at order. Pin 1 is +
Changed lines of the file:
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@@
       (effects (font (size 1.27 1.27)) (justify left) )
     )
-    (property "Value" "220uF" (at 121.92 57.66 0)
+    (property "Value" "330uF" (at 121.92 57.66 0)
       (effects (font (size 1.27 1.27)) (justify left) )
     )
-    (property "Footprint" "Capacitor_SMD:CP_Elec_16x17.5" (at 121.92 57.66 0)
+    (property "Footprint" "Capacitor_SMD:CP_Elec_16x22" (at 121.92 57.66 0)
       (effects (font (size 1.27 1.27)) (justify left) hide)
     )
@@
       (effects (font (size 1.27 1.27)) (justify left) hide)
     )
-    (property "Note" "Power-fail ride-through. With the sensor rail shed and the LEDs off the board draws about 0.35 W here, so the bank holds the rails up for roughly 70 ms -- enough to finish the block in flight and close the file. Any 220uF >=80V on a 16x17.5 land works; match in the JLC catalogue at order. Pin 1 is +" (at 121.92 57.66 0)
+    (property "Note" "Power-fail ride-through. With the sensor rail shed and the LEDs off the board draws about 0.35 W here, so the bank holds the rails up long enough to finish the block in flight and close the file. 16x22 rather than 16x17.5: the two footprints are identical in every copper and courtyard layer -- only the can is 4.5 mm taller -- so the extra 220 uF costs nothing but enclosure height. Any 330uF >=80V on a 16 mm land works; match in the JLC catalogue at order. Pin 1 is +" (at 121.92 57.66 0)
       (effects (font (size 1.27 1.27)) (justify left) hide)
     )
@@
       (effects (font (size 1.27 1.27)) (justify left) )
     )
-    (property "Value" "220uF" (at 129.54 57.66 0)
+    (property "Value" "330uF" (at 129.54 57.66 0)
       (effects (font (size 1.27 1.27)) (justify left) )
     )
-    (property "Footprint" "Capacitor_SMD:CP_Elec_16x17.5" (at 129.54 57.66 0)
+    (property "Footprint" "Capacitor_SMD:CP_Elec_16x22" (at 129.54 57.66 0)
       (effects (font (size 1.27 1.27)) (justify left) hide)
     )
@@
       (effects (font (size 1.27 1.27)) (justify left) hide)
     )
-    (property "Note" "Power-fail ride-through. With the sensor rail shed and the LEDs off the board draws about 0.35 W here, so the bank holds the rails up for roughly 70 ms -- enough to finish the block in flight and close the file. Any 220uF >=80V on a 16x17.5 land works; match in the JLC catalogue at order. Pin 1 is +" (at 129.54 57.66 0)
+    (property "Note" "Power-fail ride-through. With the sensor rail shed and the LEDs off the board draws about 0.35 W here, so the bank holds the rails up long enough to finish the block in flight and close the file. 16x22 rather than 16x17.5: the two footprints are identical in every copper and courtyard layer -- only the can is 4.5 mm taller -- so the extra 220 uF costs nothing but enclosure height. Any 330uF >=80V on a 16 mm land works; match in the JLC catalogue at order. Pin 1 is +" (at 129.54 57.66 0)
       (effects (font (size 1.27 1.27)) (justify left) hide)
     )

Commit message: Verify every part number against the live catalogue; docs now self-check
Asked to make sure the part numbers will match real parts at order time, so
all 23 in fab/bom.csv were looked up one at a time against LCSC and the
JLCPCB parts library. Two were wrong, and one of them mattered.

  C8544 for Q5 "MMBT3906" resolves to an S9018 -- an NPN, from a different
  manufacturer. Q5 is the transistor that pulls the P-FET gate in the USB
  over-voltage cutoff, and it has to be a PNP. Ordering as it stood would
  have assembled the wrong polarity and left that protection silently
  inoperative. Now C84105, verified: ST(Semtech) MMBT3906, PNP, SOT-23.

  C7975 for U9 SN74AHCT1G125DBVR resolves to an LMV324IPWRG4, a quad op-amp
  in TSSOP-14, out of stock. The generator already knew -- it carried a
  comment saying so and left the field blank -- but the fix never reached
  README section 7, which still offered the number. Now C7484, verified.

L2's inductor picked up a verified number on the way past (C340243, the
22 uH sibling of L1's C340244), so the hand-match list at order time drops
from eleven lines to nine.

Also found while re-exporting: export_fab.py returned an empty set from
through_hole_refs() when pcbnew was missing, so running it under the system
Python produced fab files that looked perfect -- BOM and CPL still agreed,
designator counts still matched -- and quietly asked JLC to assemble all
eight hand-soldered connectors. It now re-execs under KiCad's Python, and
raises rather than degrading if that cannot be found. The files are back to
170 designators.

Documents brought in line with the artefacts: the Rev A title against a Rev
B board, 84 x 74 mm in three places on a board that is 84 x 100, stale
track/via/BOM/designator counts, and the ordering-day part-count split.

gen/audit_docs.py now recomputes ten of those numbers from the .kicad_pcb,
bom.csv and fab/ and diffs them against the prose. It immediately caught a
via count I had just got wrong by hand -- 3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
Parts:
- L2: Note Same automotive series as L1 -> Same automotive series as L1. C340243 verified against the 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
Changed lines of the file:
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@@
       (effects (font (size 1.27 1.27)) hide)
     )
-    (property "Note" "Same automotive series as L1" (at 240.03 150.62 270)
+    (property "Note" "Same automotive series as L1. C340243 verified against the live JLC catalogue 2026-08-12: 22uH, 3A Isat, 8x8mm -- one part number below L1's C340244, which is the 33uH of the same series" (at 240.03 150.62 270)
       (effects (font (size 1.27 1.27)) hide)
     )
