File: can.kicad_sch (KiCad schematic)
At the start: 13 parts, among them U7 TJA1051T/3

Commit message: Schematic: make the hierarchy real; trunk layout does not decompose
The six sheets were pages, not a hierarchy: every cross-sheet connection
went by global label and no sheet declared an interface. Now the 40 nets
that actually leave a sheet carry hierarchical labels there and appear as
pins on that sheet's symbol at the root, so each block states what it
needs and what it provides. Rails stay global, since a power symbol is
global by definition and does not belong in a signal interface.

Three things had to be right for KiCad to see it, and each announced
itself: dropping both pin labels on a wired net let KiCad autoname it and
validate.py caught the rename; a label anchored 0.6 mm off its wire is a
floating label and ERC said so; and 40 and 32 are not multiples of the
1.27 mm connection grid, so every pin and stub landed off-grid until the
sheets moved to 40.64. The last one hid a real bug -- the sheet symbol
stayed at x=40 while its pins moved to 40.64, leaving them 0.64 mm off
the sheet edge and every one of them unconnected.

On the trunk layout: I measured it rather than attempting it blind, and
it does not decompose into a bounded job. Of ~98 nets, 21 have the
two-pin shape already wired, 40 cross sheets and now have hierarchical
labels, and 37 are multi-pin local nodes -- the ones a person draws as a
wire tree. A trunk needs every part on the node placed against it, but
each two-pin part sits between two different nets, so trunking one net
fixes the position its other net then has to work around. That is
schematic auto-layout, not a special case of it. Restricting to nodes
whose members all end on a rail, which is the one tractable subset, finds
6 of the 37. Six nodes is not worth the machinery, and a half-working
trunk pass would read worse than the honest grid.

Board is untouched by any of this: still 0 DRC errors, 0 unconnected.

Co-Authored-By: Claude Opus 5 <noreply@anthropic.com>
Claude-Session: https://claude.ai/code/session_01DhNbL25h25p8VFCjRfJik9
Changed lines of the file:
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@@
     (effects (font (size 1.27 1.27)) (justify left bottom))
   )
-  (global_label "CAN_TX" (shape input) (at 26.67 27.94 180) (fields_autoplaced)
+  (hierarchical_label "CAN_TX" (shape bidirectional) (at 26.67 27.94 180)
     (effects (font (size 1.27 1.27)) (justify right))
-    (property "Intersheet References" "${INTERSHEET_REFS}" (at 26.67 27.94 0)
-      (effects (font (size 1.27 1.27)) (justify left) hide)
-    )
   )
-  (global_label "CAN_RX" (shape input) (at 26.67 30.48 180) (fields_autoplaced)
+  (hierarchical_label "CAN_RX" (shape bidirectional) (at 26.67 30.48 180)
     (effects (font (size 1.27 1.27)) (justify right))
-    (property "Intersheet References" "${INTERSHEET_REFS}" (at 26.67 30.48 0)
-      (effects (font (size 1.27 1.27)) (justify left) hide)
-    )
   )
-  (global_label "CAN_S" (shape input) (at 26.67 38.1 180) (fields_autoplaced)
+  (hierarchical_label "CAN_S" (shape bidirectional) (at 26.67 38.1 180)
     (effects (font (size 1.27 1.27)) (justify right))
-    (property "Intersheet References" "${INTERSHEET_REFS}" (at 26.67 38.1 0)
-      (effects (font (size 1.27 1.27)) (justify left) hide)
-    )
   )
   (global_label "CANH_T" (shape input) (at 62.23 30.48 0) (fields_autoplaced)
@@
     )
   )
-  (global_label "CAN_S" (shape input) (at 35.56 104.14 180) (fields_autoplaced)
+  (hierarchical_label "CAN_S" (shape bidirectional) (at 35.56 104.14 180)
     (effects (font (size 1.27 1.27)) (justify right))
-    (property "Intersheet References" "${INTERSHEET_REFS}" (at 35.56 104.14 0)
-      (effects (font (size 1.27 1.27)) (justify left) hide)
-    )
   )
   (global_label "CANH_T" (shape input) (at 34.29 119.38 180) (fields_autoplaced)
@@
     )
   )
-  (global_label "CAN_H" (shape input) (at 54.61 119.38 0) (fields_autoplaced)
+  (hierarchical_label "CAN_H" (shape bidirectional) (at 54.61 119.38 0)
     (effects (font (size 1.27 1.27)) (justify left))
-    (property "Intersheet References" "${INTERSHEET_REFS}" (at 54.61 119.38 0)
-      (effects (font (size 1.27 1.27)) (justify left) hide)
-    )
   )
-  (global_label "CAN_L" (shape input) (at 54.61 124.46 0) (fields_autoplaced)
+  (hierarchical_label "CAN_L" (shape bidirectional) (at 54.61 124.46 0)
     (effects (font (size 1.27 1.27)) (justify left))
-    (property "Intersheet References" "${INTERSHEET_REFS}" (at 54.61 124.46 0)
-      (effects (font (size 1.27 1.27)) (justify left) hide)
-    )
   )
-  (global_label "CAN_H" (shape input) (at 35.56 134.62 180) (fields_autoplaced)
+  (hierarchical_label "CAN_H" (shape bidirectional) (at 35.56 134.62 180)
     (effects (font (size 1.27 1.27)) (justify right))
-    (property "Intersheet References" "${INTERSHEET_REFS}" (at 35.56 134.62 0)
-      (effects (font (size 1.27 1.27)) (justify left) hide)
-    )
   )
   (global_label "CAN_SPLIT" (shape input) (at 69.85 134.62 0) (fields_autoplaced)
@@
     )
   )
-  (global_label "CAN_L" (shape input) (at 53.34 149.86 0) (fields_autoplaced)
+  (hierarchical_label "CAN_L" (shape bidirectional) (at 53.34 149.86 0)
     (effects (font (size 1.27 1.27)) (justify left))
-    (property "Intersheet References" "${INTERSHEET_REFS}" (at 53.34 149.86 0)
-      (effects (font (size 1.27 1.27)) (justify left) hide)
-    )
   )
   (global_label "CAN_SPLIT" (shape input) (at 35.56 165.1 180) (fields_autoplaced)
@@
     )
   )
-  (global_label "CAN_H" (shape input) (at 35.56 180.34 180) (fields_autoplaced)
+  (hierarchical_label "CAN_H" (shape bidirectional) (at 35.56 180.34 180)
     (effects (font (size 1.27 1.27)) (justify right))
-    (property "Intersheet References" "${INTERSHEET_REFS}" (at 35.56 180.34 0)
-      (effects (font (size 1.27 1.27)) (justify left) hide)
-    )
   )
-  (global_label "CAN_L" (shape input) (at 35.56 195.58 180) (fields_autoplaced)
+  (hierarchical_label "CAN_L" (shape bidirectional) (at 35.56 195.58 180)
     (effects (font (size 1.27 1.27)) (justify right))
-    (property "Intersheet References" "${INTERSHEET_REFS}" (at 35.56 195.58 0)
-      (effects (font (size 1.27 1.27)) (justify left) hide)
-    )
   )
-  (global_label "CAN_H" (shape input) (at 44.45 215.9 270) (fields_autoplaced)
+  (hierarchical_label "CAN_H" (shape bidirectional) (at 44.45 215.9 270)
     (effects (font (size 1.27 1.27)) (justify right))
-    (property "Intersheet References" "${INTERSHEET_REFS}" (at 44.45 215.9 0)
-      (effects (font (size 1.27 1.27)) (justify left) hide)
-    )
   )
-  (global_label "CAN_L" (shape input) (at 44.45 237.49 270) (fields_autoplaced)
+  (hierarchical_label "CAN_L" (shape bidirectional) (at 44.45 237.49 270)
     (effects (font (size 1.27 1.27)) (justify right))
-    (property "Intersheet References" "${INTERSHEET_REFS}" (at 44.45 237.49 0)
-      (effects (font (size 1.27 1.27)) (justify left) hide)
-    )
   )
   (symbol (lib_id "Interface_CAN_LIN:TJA1051T-3") (at 44.45 33.02 0) (unit 1)
