File: can.kicad_sch (KiCad schematic)
At the start: 13 parts, among them U7 TJA1051T/3

Commit message: Power-fail ride-through: detect, coast, shed; board grows to 84 x 100
The ignition cuts this board's power with a log file open, every drive.
Three new pieces make that survivable, all simulated before layout:

- Detect: TLV431 + 100k/12.7k divider on VBAT_F, AHEAD of the ideal
  diode, asserting PWR_FAIL (IO15) at 11.0 V with ~0.3 V hysteresis.
  The harness collapses microseconds after the key turns while +VBAT
  coasts, so the warning costs no stored energy.
- Coast: two 220 uF/100 V cans join the 100 uF on +VBAT. 540 uF on the
  input rail, where a volt of headroom is worth most.
- Shed: AO3401 + 2N7002 high-side switch on the sensor rail (SENS_EN,
  IO16, off at reset), with PF1 moved behind it so a tripped sensor
  fuse can also be power-cycled from firmware.

Simulated end to end: detection <1 ms after the cut, then 108 ms to
converter dropout with sensors shed, 53 ms without -- the switch doubles
the flush budget. ISO pulse 1's brownout shortens from 8.2 to 5.6 ms.

The two cans plus the detector had no free board left on 84 x 84, so the
board grows to 84 x 100 (still JLC's cheap tier): bottom-edge furniture
and mounting holes move down 16 mm, one can per side, and the detector/
switch column gets its own placement zone. Also included from the audit:
the 3V3 buck's own input capacitor pair at its VIN pin (it was reaching
12.6 mm across to the 5 V island's), the CAN transceiver and AHCT buffer
bypasses pinned at their pins, and Power-class tracks at 0.55 mm to clear
IPC-2221 for 2 A at a 20 C rise.

Hard-won generator fix: a literal newline inside a symbol property is
accepted by KiCad's loader but silently breaks connectivity for every
symbol after it in the file -- the netlist dropped 45 components with no
error pointing anywhere near the cause. The emitter now flattens all
whitespace in property strings.

Board: 0 DRC violations, 0 unconnected, physical audit clean end to end.
185 components, 111 nets, ERC clean, netlist verified node-for-node.

Co-Authore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
Parts:
- removed C30, C31: 100nF, Capacitor_SMD:C_0805_2012Metric, symbol Device:C
- removed C32: 4.7nF, Capacitor_SMD:C_0805_2012Metric, symbol Device:C
- removed R43: 10k, Resistor_SMD:R_0805_2012Metric, symbol Device:R
- removed R44, R45: 60.4, Resistor_SMD:R_0805_2012Metric, symbol Device:R
- removed U7: TJA1051T/3, Package_SO:SOIC-8_3.9x4.9mm_P1.27mm, symbol Interface_CAN_LIN:TJA1051T-3
- added C35, C36: 100nF, Capacitor_SMD:C_0805_2012Metric, symbol Device:C
- added C37: 4.7nF, Capacitor_SMD:C_0805_2012Metric, symbol Device:C
- added R50: 10k, Resistor_SMD:R_0805_2012Metric, symbol Device:R
- added R51, R52: 60.4, Resistor_SMD:R_0805_2012Metric, symbol Device:R
- added U8: TJA1051T/3, Package_SO:SOIC-8_3.9x4.9mm_P1.27mm, symbol Interface_CAN_LIN:TJA1051T-3
Connections:
- net +3V3: now also C36.1, U8.5 (VIO)
- net +5V: now also C35.1, U8.3 (VCC)
- net CANH_T: now also U8.7 (CANH)
- net CANL_T: now also U8.6 (CANL)
- net CAN_L: now also R52.2
- net CAN_RX: now also U8.4 (RXD)
- net CAN_S: now also R50.1, U8.8 (S)
- net CAN_SPLIT: now also C37.1, R51.2, R52.1
- net CAN_TX: now also U8.1 (TXD)
- net GND: now also C35.2, C36.2, C37.2, R50.2, U8.2 (GND)
- net TERM_A: now also R51.1

Commit message: USB OVP, card-slot ESD, SD test points, and a gold-standard schematic
Hardware, all simulation- or review-driven:
- USB overvoltage cutoff: TLV431 + AO3401 + MMBT3906 series switch on
  VBUS, tripping at 5.77 V. Re-simulated: a compliant 5 V source passes
  at 4.99 V, the switch opens at 5.95 V of brick, and the +5V rail never
  exceeds 5.2 V from anything up to 14 V -- where a 9 V brick previously
  drove it to 8.4 V against the TJA1051's 6 V absolute maximum.
  Off-the-shelf OVP parts were rejected first: the TPS25200 class cuts
  off near 7 V, which is no protection for a 6 V limit.
- Two SRV05-4 arrays clamp every microSD card contact (LCSC C13612);
  until now the ESP32's ~2 kV pin diodes were all that stood behind a
  card swapped by hand after every session.
- A second USBLC6 clamps the USB-C CC pins -- the first contacts every
  plug insertion touches, previously landing on bare 5.1k resistors.
- Test points on SD_CLK and SD_CMD, the most likely scope targets at
  bring-up and otherwise reachable only on fine-pitch pads.

The schematic itself was rebuilt to read like a reference design
(RejsaCAN was the benchmark): every circuit is now a hand-drawn block --
power-fail detector, sensor-rail switch, USB OVP, connector pull-
resistor clusters, and a single utility panel for test points, ERC
flags, mounting holes and the power LED. Sentence-length values became
part numbers ("0.2A PTC", "AO3401A", "600R") with ratings kept in
hidden fields, which also answers the external review's value-hygiene
findings. Title blocks carry rev B and a date. The Power sheet shrank
from A2 back to A3 in the process.

gen/README.md now documents the whole pipeline -- stages, the block-
drawing conventions with per-rotation pin geometry, the junction rules,
and the traps (property newlines, off-grid points, anchors keeping
their natural rotation) -- so the next board reuses all of it.

Board: 84 x 100, 0 DRC violations, 0 unconnected, 0 courtyard overlaps,
physical audit clean. BOM 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
Parts:
- removed R50: 10k, Resistor_SMD:R_0805_2012Metric, symbol Device:R
- removed R51, R52: 60.4, Resistor_SMD:R_0805_2012Metric, symbol Device:R
- removed TP8: CAN_H, TestPoint:TestPoint_Pad_D1.5mm, symbol Connector:TestPoint
- removed TP9: CAN_L, TestPoint:TestPoint_Pad_D1.5mm, symbol Connector:TestPoint
- removed U8: TJA1051T/3, Package_SO:SOIC-8_3.9x4.9mm_P1.27mm, symbol Interface_CAN_LIN:TJA1051T-3
- added R54: 10k, Resistor_SMD:R_0805_2012Metric, symbol Device:R
- added R55, R56: 60.4, Resistor_SMD:R_0805_2012Metric, symbol Device:R
- added TP10: CAN_H, TestPoint:TestPoint_Pad_D1.5mm, symbol Connector:TestPoint
- added TP11: CAN_L, TestPoint:TestPoint_Pad_D1.5mm, symbol Connector:TestPoint
- added U12: TJA1051T/3, Package_SO:SOIC-8_3.9x4.9mm_P1.27mm, symbol Interface_CAN_LIN:TJA1051T-3
- L3: value 51uH CMC -> 51uH
Connections:
- net +3V3: now also U12.5 (VIO)
- net +5V: now also U12.3 (VCC)
- net CANH_T: now also U12.7 (CANH)
- net CANL_T: now also U12.6 (CANL)
- net CAN_H: now also TP10.1
- net CAN_L: now also R56.2, TP11.1
- net CAN_RX: now also U12.4 (RXD)
- net CAN_S: now also R54.1, U12.8 (S)
- net CAN_SPLIT: now also R55.2, R56.1
- net CAN_TX: now also U12.1 (TXD)
- net GND: now also R54.2, U12.2 (GND)
- net TERM_A: now also R55.1

Commit message: Studies 9-11, post-route extraction, strap audit, readable labels, production BOM numbers
New tests, run against the final board:
- audit_routes.py: Dijkstra IR drop over the routed copper (worst 55 mV
  at rated current), SD/USB/CAN routed lengths (USB pair matched to
  1.1 mm), buck switch-node copper area. All clean.
- audit_straps.py: every ESP32-S3 strapping pin against what the netlist
  hangs on it; all five boot in their required state.
- simulate.py 9, stability: the LM5164 ripple-injection criterion across
  the input window. Found the ramp thin (10.6 mV) at a legitimate 8 V
  operating point -- ramp caps changed 3.3 nF -> 2.2 nF, now 15.8 mV+
  everywhere above crank voltages. Board rebuilt: 0 DRC, 0 unconnected,
  0 overlaps.
- simulate.py 10, CAN bus: TJA1051 through the choke and split
  termination into 5 m of terminated line -- 2.00 V dominant at the far
  end, no overshoot.
- simulate.py 11, budgets: enclosure thermal for the in-dash mount
  (sealed ABS is fine in the dash, would exceed the electrolytics' 105 C
  in an engine bay -- documented), fuse derating 69 %, I2C rise time vs
  Qwiic chains, WS2812 count, SD switch drop, connector contacts.
- tolerance MC gains the ride-through corner: 36 ms at caps -20 % /
  load +40 %, still covering a healthy-card flush.

Schematic readability, second pass: net-name labels moved onto short
vertical spurs clear of the circuits (deleting them outright renames
nets to Net-(R5-Pad2) and breaks name-based verification -- now in
gen/README.md), end-labels extend away from what they feed, and the
sensor-switch block redrawn at 1.5x pitch. Reversed-5V behaviour per
connector documented in the README.

BOM production pass: verified LCSC numbers added for the TVS families,
BAT54S, MM3Z zener and 2N7002s (21 numbered lines); the 39 blank lines
are JLC-auto-matched basic R/C; the 12 extended lines that must be
hand-matched in the order UI are listed in README 11. No guessed part
numbers.

gen/README.md gains the readab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
Parts:
- D6, D7: MPN Littelfuse SMAJ26CA -> Diodes Inc SMAJ26CA-13-F
Changed lines of the file:
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@@
       (effects (font (size 1.27 1.27)) (justify left) hide)
     )
-    (property "MPN" "Littelfuse SMAJ26CA" (at 91.44 39.88 90)
+    (property "MPN" "Diodes Inc SMAJ26CA-13-F" (at 91.44 39.88 90)
       (effects (font (size 1.27 1.27)) (justify left) hide)
     )
@@
       (effects (font (size 1.27 1.27)) (justify left) hide)
     )
-    (property "MPN" "Littelfuse SMAJ26CA" (at 91.44 72.9 90)
+    (property "MPN" "Diodes Inc SMAJ26CA-13-F" (at 91.44 72.9 90)
       (effects (font (size 1.27 1.27)) (justify left) hide)
     )

Commit message: Board change: termination off by default, 0-5 V sensors by default, 2x330 uF
Three defaults changed in gen/generate_schematic.py, then the whole chain
regenerated: schematic, board, fab, plots. Schematic is ERC-clean at 206
components / 114 nets; the board rebuilt to 0 DRC violations and 0
unconnected; fab BOM and CPL agree at 178 designators.

CAN termination now ships OFF. JP1 moves from SolderJumper-2_Bridged to
_Open. The board was shipping terminated, matching the Autosport Labs
convention, but the common case here is plugging into a vehicle bus that
is already terminated at both ends — where a third 120 ohm takes the pair
to about 40 ohm and can stop the bus working. Defaulting on made that an
easy mistake; defaulting off means there is nothing to remember before
plugging into a car, and bridging JP1 is a deliberate act for a bench bus
where this board is an end node.

Analog channels now ship in the 0-5 V range. The four RANGE jumpers move
from SolderJumper-3_Open to _Bridged12, closing the 15k leg. They were
shipping fully open, which is no divider at all, so a 5 V sensor needed a
jumper somebody had to remember to fit — and the firmware's DIVIDER_GAIN
of 1.7334 assumed the 0-5 V ratio, so an unfitted jumper read 73 % high.
Board and firmware defaults now agree out of the box.

Ride-through bank 540 -> 760 uF. C6/C7 go 220 -> 330 uF in CP_Elec_16x22.
That footprint is identical to the 16x17.5 it replaces in every copper,
courtyard, silk and fab layer — only the 3D can is 4.5 mm taller — so the
extra 220 uF costs nothing but enclosure height, and the routed board did
not have to move for it.

It is not free everywhere: inrush I2t is linear in C, so the 2 A fuse's
margin drops from ~5x to ~3.6x. Noted in the generator next to the value
so the next person to grow the bank sees it.

ngspice is not installed here, so the new hold-up figures (152 / 75 ms,
from 108 / 53) are SCALED, not measured — hold-up is linear in C for a
constant-power load over a fixed window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
Parts:
- JP1: value TERM (default ON) -> TERM (default OFF); footprint Jumper:SolderJumper-2_P1.3mm_Bridged_Pad1.0x1.5mm -> Jumper:SolderJumper-2_P1.3mm_Open_Pad1.0x1.5mm; symbol Jumper:SolderJumper_2_Bridged -> Jumper:SolderJumper_2_Open; Note Cut the trace to remove the 120 ohm termination on a mid-bu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 -> Ships OPEN: unterminated. Bridge the pads only when this bo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
Changed lines of the file:
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@@
     )
   )
-  (symbol (lib_id "Jumper:SolderJumper_2_Bridged") (at 100.33 38.1 270) (unit 1)
+  (symbol (lib_id "Jumper:SolderJumper_2_Open") (at 100.33 38.1 270) (unit 1)
     (in_bom yes) (on_board yes) (dnp no)
     (property "Reference" "JP1" (at 101.6 36.83 90)
       (effects (font (size 1.27 1.27)) (justify left) )
     )
-    (property "Value" "TERM (default ON)" (at 101.6 39.88 90)
+    (property "Value" "TERM (default OFF)" (at 101.6 39.88 90)
       (effects (font (size 1.27 1.27)) (justify left) )
     )
-    (property "Footprint" "Jumper:SolderJumper-2_P1.3mm_Bridged_Pad1.0x1.5mm" (at 101.6 39.88 90)
+    (property "Footprint" "Jumper:SolderJumper-2_P1.3mm_Open_Pad1.0x1.5mm" (at 101.6 39.88 90)
       (effects (font (size 1.27 1.27)) (justify left) hide)
     )
@@
       (effects (font (size 1.27 1.27)) (justify left) hide)
     )
-    (property "Note" "Cut the trace to remove the 120 ohm termination on a mid-bus node" (at 101.6 39.88 90)
+    (property "Note" "Ships OPEN: unterminated. Bridge the pads only when this board is an END node on its own bus. A vehicle's bus -- OBD-II diagnostics included -- is already terminated at both ends, and a third 120 ohm across the pair takes it to about 40 ohm and can stop it working. Defaulting terminated made that an easy mistake to make" (at 101.6 39.88 90)
       (effects (font (size 1.27 1.27)) (justify left) hide)
     )
