File: analog.kicad_sch (KiCad schematic)
At the start: 51 parts, among them J10 Sensor harness, U13 ADS1115

Commit message: Board change: termination off by default, 0-5 V sensors by default, 2x330 uF
Three defaults changed in gen/generate_schematic.py, then the whole chain
regenerated: schematic, board, fab, plots. Schematic is ERC-clean at 206
components / 114 nets; the board rebuilt to 0 DRC violations and 0
unconnected; fab BOM and CPL agree at 178 designators.

CAN termination now ships OFF. JP1 moves from SolderJumper-2_Bridged to
_Open. The board was shipping terminated, matching the Autosport Labs
convention, but the common case here is plugging into a vehicle bus that
is already terminated at both ends — where a third 120 ohm takes the pair
to about 40 ohm and can stop the bus working. Defaulting on made that an
easy mistake; defaulting off means there is nothing to remember before
plugging into a car, and bridging JP1 is a deliberate act for a bench bus
where this board is an end node.

Analog channels now ship in the 0-5 V range. The four RANGE jumpers move
from SolderJumper-3_Open to _Bridged12, closing the 15k leg. They were
shipping fully open, which is no divider at all, so a 5 V sensor needed a
jumper somebody had to remember to fit — and the firmware's DIVIDER_GAIN
of 1.7334 assumed the 0-5 V ratio, so an unfitted jumper read 73 % high.
Board and firmware defaults now agree out of the box.

Ride-through bank 540 -> 760 uF. C6/C7 go 220 -> 330 uF in CP_Elec_16x22.
That footprint is identical to the 16x17.5 it replaces in every copper,
courtyard, silk and fab layer — only the 3D can is 4.5 mm taller — so the
extra 220 uF costs nothing but enclosure height, and the routed board did
not have to move for it.

It is not free everywhere: inrush I2t is linear in C, so the 2 A fuse's
margin drops from ~5x to ~3.6x. Noted in the generator next to the value
so the next person to grow the bank sees it.

ngspice is not installed here, so the new hold-up figures (152 / 75 ms,
from 108 / 53) are SCALED, not measured — hold-up is linear in C for a
constant-power load over a fixed window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
Parts:
- JP10: value RANGE3 -> RANGE3 (default 0-5V); footprint Jumper:SolderJumper-3_P1.3mm_Open_Pad1.0x1.5mm -> Jumper:SolderJumper-3_P1.3mm_Bridged12_Pad1.0x1.5mm; symbol Jumper:SolderJumper_3_Open -> Jumper:SolderJumper_3_Bridged12; Note C-A = 0-5V range, C-B = 0-16V range, both open = no divider -> Ships BRIDGED 1-2 = the 0-5V range, which is what almost ev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
- JP13: value RANGE4 -> RANGE4 (default 0-5V); footprint Jumper:SolderJumper-3_P1.3mm_Open_Pad1.0x1.5mm -> Jumper:SolderJumper-3_P1.3mm_Bridged12_Pad1.0x1.5mm; symbol Jumper:SolderJumper_3_Open -> Jumper:SolderJumper_3_Bridged12; Note C-A = 0-5V range, C-B = 0-16V range, both open = no divider -> Ships BRIDGED 1-2 = the 0-5V range, which is what almost ev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
- JP4: value RANGE1 -> RANGE1 (default 0-5V); footprint Jumper:SolderJumper-3_P1.3mm_Open_Pad1.0x1.5mm -> Jumper:SolderJumper-3_P1.3mm_Bridged12_Pad1.0x1.5mm; symbol Jumper:SolderJumper_3_Open -> Jumper:SolderJumper_3_Bridged12; Note C-A = 0-5V range, C-B = 0-16V range, both open = no divider -> Ships BRIDGED 1-2 = the 0-5V range, which is what almost ev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
- JP7: value RANGE2 -> RANGE2 (default 0-5V); footprint Jumper:SolderJumper-3_P1.3mm_Open_Pad1.0x1.5mm -> Jumper:SolderJumper-3_P1.3mm_Bridged12_Pad1.0x1.5mm; symbol Jumper:SolderJumper_3_Open -> Jumper:SolderJumper_3_Bridged12; Note C-A = 0-5V range, C-B = 0-16V range, both open = no divider -> Ships BRIDGED 1-2 = the 0-5V range, which is what almost ev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
Changed lines of the file:
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@@
     )
   )
-  (symbol (lib_id "Jumper:SolderJumper_3_Open") (at 87.63 91.44 180) (unit 1)
+  (symbol (lib_id "Jumper:SolderJumper_3_Bridged12") (at 87.63 91.44 180) (unit 1)
     (in_bom yes) (on_board yes) (dnp no)
     (property "Reference" "JP4" (at 87.63 72.39 0)
       (effects (font (size 1.27 1.27)) )
     )
-    (property "Value" "RANGE1" (at 87.63 93.47 0)
-      (effects (font (size 1.27 1.27)) )
-    )
-    (property "Footprint" "Jumper:SolderJumper-3_P1.3mm_Open_Pad1.0x1.5mm" (at 87.63 93.47 0)
+    (property "Value" "RANGE1 (default 0-5V)" (at 87.63 93.47 0)
+      (effects (font (size 1.27 1.27)) )
+    )
+    (property "Footprint" "Jumper:SolderJumper-3_P1.3mm_Bridged12_Pad1.0x1.5mm" (at 87.63 93.47 0)
       (effects (font (size 1.27 1.27)) hide)
     )
@@
       (effects (font (size 1.27 1.27)) hide)
     )
-    (property "Note" "C-A = 0-5V range, C-B = 0-16V range, both open = no divider" (at 87.63 93.47 0)
+    (property "Note" "Ships BRIDGED 1-2 = the 0-5V range, which is what almost every automotive sensor is. Cut 1-2 and bridge 2-3 for 0-16V; cut 1-2 and leave both open for no divider (then close BYPASS1 for a raw 0-3.3V sensor). Defaulting to 0-5V also means the firmware's DIVIDER_GAIN matches the board as shipped" (at 87.63 93.47 0)
       (effects (font (size 1.27 1.27)) hide)
     )
@@
     )
   )
-  (symbol (lib_id "Jumper:SolderJumper_3_Open") (at 87.63 163.83 180) (unit 1)
+  (symbol (lib_id "Jumper:SolderJumper_3_Bridged12") (at 87.63 163.83 180) (unit 1)
     (in_bom yes) (on_board yes) (dnp no)
     (property "Reference" "JP7" (at 87.63 144.78 0)
       (effects (font (size 1.27 1.27)) )
     )
-    (property "Value" "RANGE2" (at 87.63 165.86 0)
-      (effects (font (size 1.27 1.27)) )
-    )
-    (property "Footprint" "Jumper:SolderJumper-3_P1.3mm_Open_Pad1.0x1.5mm" (at 87.63 165.86 0)
+    (property "Value" "RANGE2 (default 0-5V)" (at 87.63 165.86 0)
+      (effects (font (size 1.27 1.27)) )
+    )
+    (property "Footprint" "Jumper:SolderJumper-3_P1.3mm_Bridged12_Pad1.0x1.5mm" (at 87.63 165.86 0)
       (effects (font (size 1.27 1.27)) hide)
     )
@@
       (effects (font (size 1.27 1.27)) hide)
     )
-    (property "Note" "C-A = 0-5V range, C-B = 0-16V range, both open = no divider" (at 87.63 165.86 0)
+    (property "Note" "Ships BRIDGED 1-2 = the 0-5V range, which is what almost every automotive sensor is. Cut 1-2 and bridge 2-3 for 0-16V; cut 1-2 and leave both open for no divider (then close BYPASS2 for a raw 0-3.3V sensor). Defaulting to 0-5V also means the firmware's DIVIDER_GAIN matches the board as shipped" (at 87.63 165.86 0)
       (effects (font (size 1.27 1.27)) hide)
     )
@@
     )
   )
-  (symbol (lib_id "Jumper:SolderJumper_3_Open") (at 87.63 236.22 180) (unit 1)
+  (symbol (lib_id "Jumper:SolderJumper_3_Bridged12") (at 87.63 236.22 180) (unit 1)
     (in_bom yes) (on_board yes) (dnp no)
     (property "Reference" "JP10" (at 87.63 217.17 0)
       (effects (font (size 1.27 1.27)) )
     )
-    (property "Value" "RANGE3" (at 87.63 238.25 0)
-      (effects (font (size 1.27 1.27)) )
-    )
-    (property "Footprint" "Jumper:SolderJumper-3_P1.3mm_Open_Pad1.0x1.5mm" (at 87.63 238.25 0)
+    (property "Value" "RANGE3 (default 0-5V)" (at 87.63 238.25 0)
+      (effects (font (size 1.27 1.27)) )
+    )
+    (property "Footprint" "Jumper:SolderJumper-3_P1.3mm_Bridged12_Pad1.0x1.5mm" (at 87.63 238.25 0)
       (effects (font (size 1.27 1.27)) hide)
     )
@@
       (effects (font (size 1.27 1.27)) hide)
     )
-    (property "Note" "C-A = 0-5V range, C-B = 0-16V range, both open = no divider" (at 87.63 238.25 0)
+    (property "Note" "Ships BRIDGED 1-2 = the 0-5V range, which is what almost every automotive sensor is. Cut 1-2 and bridge 2-3 for 0-16V; cut 1-2 and leave both open for no divider (then close BYPASS3 for a raw 0-3.3V sensor). Defaulting to 0-5V also means the firmware's DIVIDER_GAIN matches the board as shipped" (at 87.63 238.25 0)
       (effects (font (size 1.27 1.27)) hide)
     )
@@
     )
   )
-  (symbol (lib_id "Jumper:SolderJumper_3_Open") (at 214.63 52.07 180) (unit 1)
+  (symbol (lib_id "Jumper:SolderJumper_3_Bridged12") (at 214.63 52.07 180) (unit 1)
     (in_bom yes) (on_board yes) (dnp no)
     (property "Reference" "JP13" (at 214.63 33.02 0)
       (effects (font (size 1.27 1.27)) )
     )
-    (property "Value" "RANGE4" (at 214.63 54.1 0)
-      (effects (font (size 1.27 1.27)) )
-    )
-    (property "Footprint" "Jumper:SolderJumper-3_P1.3mm_Open_Pad1.0x1.5mm" (at 214.63 54.1 0)
+    (property "Value" "RANGE4 (default 0-5V)" (at 214.63 54.1 0)
+      (effects (font (size 1.27 1.27)) )
+    )
+    (property "Footprint" "Jumper:SolderJumper-3_P1.3mm_Bridged12_Pad1.0x1.5mm" (at 214.63 54.1 0)
       (effects (font (size 1.27 1.27)) hide)
     )
@@
       (effects (font (size 1.27 1.27)) hide)
     )
-    (property "Note" "C-A = 0-5V range, C-B = 0-16V range, both open = no divider" (at 214.63 54.1 0)
-      (effects (font (size 1.27 1.27)) hide)
-    )
+    (property "Note" "Ships BRIDGED 1-2 = the 0-5V range, which is what almost every automotive sensor is. Cut 1-2 and bridge 2-3 for 0-16V; cut 1-2 and leave both open for no divider (then close BYPASS4 for a raw 0-3.3V sensor). Defaulting to 0-5V also means the firmware's DIVIDER_GAIN matches the board as shipped" (at 214.63 54.1 0)
+      (effects (font (size 1.27 1.27)) hide)
+    )
